Commit message: create custom hardware interface

File: src/rpi_diff_hw_control-main/description/urdf/robot_core.xacro (robot description, xacro)
@@ -25,18 +25,18 @@
     <link name="chassis">
         <visual>
-            <origin xyz="0.075 0 0.03"/>
+            <origin xyz="0.15 0 0.075"/>
             <geometry>
-                <box size="0.15 0.19 0.06"/>
+                <box size="0.3 0.3 0.15"/>
             </geometry>
             <material name="orange"/>
         </visual>
         <collision>
-            <origin xyz="0.075 0 0.03"/>
+            <origin xyz="0.15 0 0.075"/>
             <geometry>
-                <box size="0.15 0.19 0.06"/>
+                <box size="0.3 0.3 0.15"/>
             </geometry>
         </collision>
-        <xacro:inertial_box mass="0.8" x="0.15" y="0.19" z="0.06">
-            <origin xyz="0.075 0 0.06" rpy="0 0 0"/>
+        <xacro:inertial_box mass="0.5" x="0.3" y="0.3" z="0.15">
+            <origin xyz="0.15 0 0.075" rpy="0 0 0"/>
         </xacro:inertial_box>
     </link>
@@ -45,5 +45,5 @@
         <parent link="base_link"/>
         <child link="left_wheel"/>
-        <origin xyz="0 0.065 0" rpy="-${pi/2} 0 0" />
+        <origin xyz="0 0.175 0" rpy="-${pi/2} 0 0" />
         <axis xyz="0 0 1"/>
     </joint>
@@ -51,5 +51,5 @@
         <visual>
             <geometry>
-                <cylinder radius="0.0325" length="0.025"/>
+                <cylinder radius="0.05" length="0.04"/>
             </geometry>
             <material name="black"/>
@@ -57,8 +57,8 @@
         <collision>
             <geometry>
-                <cylinder radius="0.0325" length="0.025"/>
+                <cylinder radius="0.05" length="0.04"/>
             </geometry>
         </collision>
-        <xacro:inertial_cylinder mass="0.038" length="0.025" radius="0.0325">
+        <xacro:inertial_cylinder mass="0.1" length="0.04" radius="0.05">
             <origin xyz="0 0 0" rpy="0 0 0"/>
         </xacro:inertial_cylinder>
@@ -68,5 +68,5 @@
         <parent link="base_link"/>
         <child link="right_wheel"/>
-        <origin xyz="0 -0.065 0" rpy="${pi/2} 0 0" />
+        <origin xyz="0 -0.175 0" rpy="${pi/2} 0 0" />
         <axis xyz="0 0 -1"/>
     </joint>
@@ -74,5 +74,5 @@
         <visual>
             <geometry>
-                <cylinder radius="0.0325" length="0.025"/>
+                <cylinder radius="0.05" length="0.04"/>
             </geometry>
             <material name="black"/>
@@ -80,8 +80,8 @@
         <collision>
             <geometry>
-                <cylinder radius="0.0325" length="0.025"/>
+                <cylinder radius="0.05" length="0.04"/>
             </geometry>
         </collision>
-        <xacro:inertial_cylinder mass="0.038" length="0.025" radius="0.0325">
+        <xacro:inertial_cylinder mass="0.1" length="0.04" radius="0.05">
             <origin xyz="0 0 0" rpy="0 0 0"/>
         </xacro:inertial_cylinder>
@@ -91,10 +91,10 @@
         <parent link="chassis"/>
         <child link="caster_wheel"/>
-        <origin xyz="0.08 0 0"/>
+        <origin xyz="0.24 0 0"/>
     </joint>
     <link name="caster_wheel">
         <visual>
             <geometry>
-                <sphere radius="0.007"/>
+                <sphere radius="0.05"/>
             </geometry>
             <material name="blue"/>
@@ -102,8 +102,8 @@
         <collision>
             <geometry>
-                <sphere radius="0.007"/>
+                <sphere radius="0.05"/>
             </geometry>
         </collision>
-        <xacro:inertial_sphere mass="0.1" radius="0.007">
+        <xacro:inertial_sphere mass="0.1" radius="0.05">
             <origin xyz="0 0 0" rpy="0 0 0"/>
         </xacro:inertial_sphere>
